File: Dongle Production Files/XBee-Explorer-Dongle-GiantPanel-v21.brd (EAGLE design)
At the start: 241.8 x 155.4 mm, 743 parts, among them U1 MIC5205 3.3V, U10 MIC5205 3.3V, U11 FT231XS, U12 XBEE-1B3, U13 MIC5205 3.3V, U14 FT231XS, U15 XBEE-1B3, U16 MIC5205 3.3V, U17 FT231XS, U18 XBEE-1B3, U19 MIC5205 3.3V, U2 XBEE-1B3, U20 FT231XS, U21 XBEE-1B3, U22 MIC5205 3.3V, U23 FT231XS, U24 XBEE-1B3, U25 MIC5205 3.3V, U26 FT231XS, U27 XBEE-1B3, U28 MIC5205 3.3V, U29 FT231XS, U3 MIC5205 3.3V, U30 XBEE-1B3, U31 MIC5205 3.3V, U32 FT231XS, U33 XBEE-1B3, U34 MIC5205 3.3V, U35 FT231XS, U36 XBEE-1B3, U37 MIC5205 3.3V, U38 FT231XS, U39 XBEE-1B3, U4 FT231XS, U40 MIC5205 3.3V, U41 FT231XS, U42 XBEE-1B3, U43 MIC5205 3.3V, U44 FT231XS, U45 XBEE-1B3, U46 MIC5205 3.3V, U47 FT231XS, U48 XBEE-1B3, U49 MIC5205 3.3V, U5 FT231XS, U50 FT231XS, U51 XBEE-1B3, U52 MIC5205 3.3V, U53 FT231XS, U54 XBEE-1B3, U55 MIC5205 3.3V, U56 FT231XS, U57 XBEE-1B3, U58 MIC5205 3.3V, U59 FT231XS, U6 XBEE-1B3, U60 XBEE-1B3, U7 MIC5205 3.3V, U8 FT231XS, U9 XBEE-1B3

Commit message: re-created dongle giant panel
Parts:
- removed E$6: (no value), SparkFun-Aesthetics:FIDUCIAL-1X2
- added E$7: (no value), SparkFun-Aesthetics:FIDUCIAL-1X2
- moved E$5 134.2 mm to (232.3, 9.40), turned to 0 degrees
- moved JP12 7.62 mm to (189.2, 20.8)
- moved JP24 7.62 mm to (189.2, 49.3)
- moved JP36 7.62 mm to (189.2, 77.7)
- moved JP48 7.62 mm to (189.2, 106.2)
- moved JP60 7.62 mm to (189.2, 134.6)
- moved JP21 6.35 mm to (133.3, 49.3)
- moved JP33 6.35 mm to (133.3, 77.7)
- moved JP45 6.35 mm to (133.3, 106.2)
- moved JP57 6.35 mm to (133.3, 134.6)
- moved JP9 6.35 mm to (133.3, 20.8)
- moved C115 5.08 mm to (208.3, 129.5)
- moved C117 5.08 mm to (221.0, 133.3)
- moved C118 5.08 mm to (221.0, 139.7)
- moved C119 5.08 mm to (199.4, 136.7)
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Other:
- board size 241.8 x 155.4 mm -> 236.7 x 155.4 mm
- board text added: "Route Out"
